File: donutDriver/donutDriver.kicad_pcb (KiCad board)
At the start: 2 copper layers, 13 x 19 mm, 42 parts, among them J1 Keystone 7767, J2 Keystone 7767, J3 Keystone 7767, J4 Keystone 7767, J5 Keystone 7767, J6 Conn_Coaxial_Small, J7 Conn_Coaxial_Small, Q1 IPP320N20N3, Q2 BSS138

Commit message: begin pcb
Parts:
- C10, C11, C12, C8, C9: footprint Capacitor_THT:C_Disc_D7.5mm_W4.4mm_P5.00mm -> donutlib:TDK_Disc_D7.5mm_W5.0mm_P7.50mm
- moved H2 98.2 mm to (176.5, 145.5)
- moved H4 88.7 mm to (176.5, 73.5)
- moved J5 72.4 mm to (150.0, 142.0)
- moved J4 71.5 mm to (139.0, 141.5)
- moved J3 71.5 mm to (126.7, 142.0)
- moved J1 67.0 mm to (161.0, 59.0)
- moved H1 64.4 mm to (104.5, 145.5)
- moved C11 50.1 mm to (142.0, 68.8), turned to -90 degrees
- moved RV1 49.0 mm to (104.0, 129.5), turned to 180 degrees
- moved C12 42.0 mm to (124.0, 68.8), turned to -90 degrees
- moved Q2 38.8 mm to (116.0, 133.5)
- moved C9 38.8 mm to (136.0, 68.8), turned to -90 degrees
- moved C13 37.2 mm to (127.5, 81.5), turned to -90 degrees
- moved Q1 34.4 mm to (143.5, 82.5), turned to 180 degrees
- moved C8 30.8 mm to (130.0, 68.8), turned to -90 degrees
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Other:
- board size 13 x 19 mm -> 81 x 100 mm

Commit message: add fan switching regulator and jumpers
Parts:
- removed H1, H2, H3, H4: MountingHole, donutlib:WA-SMSI_9774025360
- removed J4, J5: Keystone 7767, donutlib:KEYSTONE_7767
- added C20: 10uF, Capacitor_SMD:C_0805_2012Metric, F.Cu at (157.7, 115.1)
- added C21: 10uF, Capacitor_SMD:C_0805_2012Metric, F.Cu at (157.7, 118.1)
- added C22: 10uF, Capacitor_SMD:C_0805_2012Metric, F.Cu at (157.7, 121.2)
- added C23: 10uF, Capacitor_SMD:C_0805_2012Metric, F.Cu at (157.7, 124.2)
- added C24: 10uF, Capacitor_SMD:C_0805_2012Metric, F.Cu at (157.7, 127.2)
- added C26: 4.7uF, Capacitor_SMD:C_1210_3225Metric, F.Cu at (156.1, 138.1)
- added C27: 1uF, Capacitor_SMD:C_0603_1608Metric, F.Cu at (151.2, 131.1)
- added J8: Conn_01x03_Pin, donutlib:CONN3_2601-3103_WAG, F.Cu at (137.5, 142.0)
- added JP1: SolderJumper_2_Open, Jumper:SolderJumper-2_P1.3mm_Open_RoundedPad1.0x1.5mm, F.Cu at (157.3, 107.0)
- added JP10: SolderJumper_2_Open, Jumper:SolderJumper-2_P1.3mm_Open_RoundedPad1.0x1.5mm, F.Cu at (166.0, 127.5)
- added JP11: SolderJumper_2_Open, Jumper:SolderJumper-2_P1.3mm_Open_RoundedPad1.0x1.5mm, F.Cu at (170.3, 113.3)
- added JP12: SolderJumper_2_Open, Jumper:SolderJumper-2_P1.3mm_Open_RoundedPad1.0x1.5mm, F.Cu at (170.3, 116.9)
- added JP13: SolderJumper_2_Open, Jumper:SolderJumper-2_P1.3mm_Open_RoundedPad1.0x1.5mm, F.Cu at (170.3, 120.5)
- added JP14: SolderJumper_2_Open, Jumper:SolderJumper-2_P1.3mm_Open_RoundedPad1.0x1.5mm, F.Cu at (170.3, 124.0)
- added JP2: SolderJumper_2_Open, Jumper:SolderJumper-2_P1.3mm_Open_RoundedPad1.0x1.5mm, F.Cu at (161.7, 116.9)
- added JP3: SolderJumper_2_Open, Jumper:SolderJumper-2_P1.3mm_Open_RoundedPad1.0x1.5mm, F.Cu at (161.7, 120.5)
- added JP4: SolderJumper_2_Open, Jumper:SolderJumper-2_P1.3mm_Open_RoundedPad1.0x1.5mm, F.Cu at (161.7, 124.0)
- added JP5: SolderJumper_2_Open, Jumper:SolderJumper-2_P1.3mm_Open_RoundedPad1.0x1.5mm, F.Cu at (161.7, 127.5)
- added JP6: SolderJumper_2_Open, Jumper:SolderJumper-2_P1.3mm_Open_RoundedPad1.0x1.5mm, F.Cu at (166.0, 113.3)
- added JP7: SolderJumper_2_Open, Jumper:SolderJumper-2_P1.3mm_Open_RoundedPad1.0x1.5mm, F.Cu at (166.0, 116.9)
- added JP8: SolderJumper_2_Open, Jumper:SolderJumper-2_P1.3mm_Open_RoundedPad1.0x1.5mm, F.Cu at (166.0, 120.5)
- added JP9: SolderJumper_2_Open, Jumper:SolderJumper-2_P1.3mm_Open_RoundedPad1.0x1.5mm, F.Cu at (166.0, 124.0)
- added M1: MountingHole_Pad, donutlib:WA-SMSI_9774025360, F.Cu at (104.5, 73.5)
- added M2: MountingHole_Pad, donutlib:WA-SMSI_9774025360, F.Cu at (176.5, 73.5)
- added M3: MountingHole_Pad, donutlib:WA-SMSI_9774025360, F.Cu at (104.5, 145.5)
- added M4: MountingHole_Pad, donutlib:WA-SMSI_9774025360, F.Cu at (176.5, 145.5)
- added R10: 10k, Resistor_SMD:R_0603_1608Metric, F.Cu at (151.2, 136.1)
- added R11: Rt, Resistor_SMD:R_0603_1608Metric, F.Cu at (151.2, 138.6)
- added R7: 10, Resistor_SMD:R_2512_6332Metric, F.Cu at (121.0, 87.0)
- added R8: 0, Resistor_SMD:R_1206_3216Metric, F.Cu at (125.5, 93.0)
- added R9: 10k, Resistor_SMD:R_0603_1608Metric, F.Cu at (151.2, 133.6)
- added RV2: 100k, Potentiometer_THT:Potentiometer_Bourns_PTV09A-2_Single_Horizontal, F.Cu at (176.6, 133.0)
- added U1: TPSM33615FRDNR, donutlib:RDN0011A-MFG, F.Cu at (156.5, 133.0)
- J3: value Keystone 7767 -> Conn_01x04_Pin; footprint donutlib:KEYSTONE_7767 -> Connector_JST:JST_XH_B4B-XH-A_1x04_P2.50mm_Vertical
- moved J7 47.2 mm to (128.0, 144.0)
- moved J3 30.8 mm to (157.2, 145.5)
- moved J6 11.5 mm to (105.0, 104.0)
- moved C10 2.00 mm to (116.0, 68.8)
- moved C11 2.00 mm to (140.0, 68.8)
- moved C12 2.00 mm to (122.0, 68.8)
- moved C8 2.00 mm to (128.0, 68.8)
- moved C9 2.00 mm to (134.0, 68.8)
Connections:
- C10 pad 2: Net-(C10-Pad2) -> Net-(JP9-B)
- C11 pad 2: Net-(C10-Pad2) -> Net-(JP10-B)
- C12 pad 2: Net-(C10-Pad2) -> Net-(JP6-B)
- C13 pad 1: Net-(C10-Pad2) -> Net-(JP10-A)
- C13 pad 2: GND -> Net-(JP1-B)
- C14 pad 1: Net-(C10-Pad2) -> Net-(JP10-A)
- C14 pad 2: GND -> Net-(JP2-B)
- C15 pad 1: Net-(C10-Pad2) -> Net-(JP10-A)
- C15 pad 2: GND -> Net-(JP3-B)
- C16 pad 1: Net-(C10-Pad2) -> Net-(JP10-A)
- C16 pad 2: GND -> Net-(JP4-B)
- C17 pad 1: Net-(C10-Pad2) -> Net-(JP10-A)
- C17 pad 2: GND -> Net-(JP5-B)
- C19 pad 1: /Gate -> Net-(J7-In)
- C7 pad 2: GND -> Net-(JP11-B)
- C8 pad 2: Net-(C10-Pad2) -> Net-(JP7-B)
- C9 pad 2: Net-(C10-Pad2) -> Net-(JP8-B)
- D2 pad 2: /Gate -> Net-(D2-A2)
- J7 pad 1: /Gate -> Net-(J7-In)
- R1 pad 1: Net-(C10-Pad2) -> Net-(JP12-A)
- R1 pad 2: /Gate -> Net-(J7-In)
- R2 pad 1: Net-(C10-Pad2) -> Net-(JP12-B)
- R2 pad 2: /Gate -> Net-(J7-In)
- R3 pad 2: Net-(C10-Pad2) -> Net-(JP12-B)
